File: hardware/rpi-pico-debugger-shoe/rpi-pico-debugger-shoe.kicad_pcb (KiCad board)
At the start: 2 copper layers, 25.4 x 54.5 mm, 49 parts, among them J1 10118193-0001LF, J2 Conn_01x02, J3 Conn_01x03, J4 Conn_01x18, J5 Conn_01x20, J6 Conn_01x03, J7 Conn_01x03, J8 Conn_01x02, SW1 PTS810_SJK_250_SMTR_LFS, U1 RP2040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

Commit message: Update libraries for KiCad 7.0
Other:
- net class Default removed
- net class Power removed
- net class USB Data removed
